File: boards/main/layout/layout.kicad_pcb (KiCad board)
At the start: 4 copper layers, 100 x 80 mm, 122 parts, among them J1 61301021121, J10 SJ1-3523N, J11 61300211121, J12 61300211121, J13 61300811121, J14 61300811121, J15 61300811121, J16 61300811121, J17 USB4085-GF-A, J2 connector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

Commit message: fixes
Parts:
- removed J17: USB4085-GF-A, USB_C_Receptacle_GCT_USB4085
- R1, R2, R3, R4: value ERJ-3EKF4701V -> ERJ-2RKF4701X; footprint R_0603_1608Metric -> R_0402_1005Metric
- R10, R9: value ERJ-2RKF1201X -> ERJ-2RKF1001X
- R7, R8: value ERJ-2RKF5101X -> ERJ-2RKF1201X
- moved R11 73.0 mm to (95.0, 84.0)
- moved R7 57.7 mm to (87.0, 66.0)
- moved R9 53.3 mm to (36.0, 41.0)
- moved R17 27.2 mm to (79.0, 88.0)
- moved R10 25.5 mm to (105.0, 84.0)
- moved R21 24.7 mm to (81.0, 84.0)
- moved C28 24.1 mm to (107.0, 80.0)
- moved C3 23.3 mm to (93.0, 38.0)
- moved R25 22.0 mm to (40.0, 61.0)
- moved R20 19.7 mm to (79.0, 86.0)
- moved C9 18.1 mm to (36.0, 39.0)
- moved R22 18.0 mm to (85.0, 84.0)
- moved C8 16.5 mm to (85.0, 58.0)
- moved C13 16.1 mm to (107.0, 48.0)
- moved R1 16.1 mm to (89.0, 28.0)
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Connections:
- R10 pad 1: SUM_FB_B -> MUX2_X_OUT
- R10 pad 2: SUM_B -> MUX1_X_FILT
- R11 pad 1: VBUS -> MUX2_Y_OUT
- R11 pad 2: LED_STAT -> MUX1_Y_FILT
- R7 pad 1: CC1 -> SUM_FB_A
- R7 pad 2: DGND -> SUM_A
- R8 pad 1: CC2 -> SUM_FB_B
- R8 pad 2: DGND -> SUM_B
- R9 pad 1: SUM_FB_A -> VBUS
- R9 pad 2: SUM_A -> LED_STAT
- U1 pad 21: NC_5V -> VBUS
- U1 pad 25: USB_DN -> NC_GPIO19
- U1 pad 26: USB_DP -> NC_GPIO20
- U10 pad 1: NC_MUX2_Y1 -> AGND
- U10 pad 11: NC_MUX2_X3 -> AGND
- U10 pad 13: NC_MUX2_X0 -> AGND
- U10 pad 14: NC_MUX2_X1 -> AGND
- U10 pad 2: NC_MUX2_Y0 -> AGND
- U10 pad 5: NC_MUX2_Y3 -> AGND
Other:
- board text removed: "USB"

Commit message: layout changes
Parts:
- added C62: GRM188Z71A106KA73D, C_0603_1608Metric, F.Cu at (91.0, 32.0)
- added C63: GCM155R71H104KE02D, C_0402_1005Metric, F.Cu at (89.0, 34.0)
- added R28: ERJ-2RKF1002X, R_0402_1005Metric, F.Cu at (40.0, 61.0)
- added R29: ERJ-2RKF1002X, R_0402_1005Metric, F.Cu at (79.0, 52.0)
- added R30: ERJ-2RKF1002X, R_0402_1005Metric, F.Cu at (95.0, 50.0)
- added R31: ERJ-2RKF1003X, R_0402_1005Metric, F.Cu at (72.0, 41.0)
- added R32: ERJ-2RKF1003X, R_0402_1005Metric, F.Cu at (60.0, 39.0)
- C31: value GCM155R71H104KE02D -> capacitor; footprint C_0402_1005Metric -> C_0805_2012Metric
- C32: value GRM188Z71A106KA73D -> GCM155R71H104KE02D; footprint C_0603_1608Metric -> C_0402_1005Metric
- R11, R12: value ERJ-2RKF1001X -> ERJ-2RKF33R0X
- R14: value ERJ-2RKF4701X -> ERJ-2RKF1001X
- R17: value ERJ-2RKF1002X -> ERJ-2RKF4701X
- R18, R19: value ERJ-2RKF1002X -> ERJ-2RKF1001X
- R26, R27: value ERJ-2RKF1003X -> ERJ-2RKF1002X
- R7: value ERJ-2RKF1201X -> ERJ-2RKF33R0X
- R9: value ERJ-2RKF1001X -> ERJ-2RKF1201X
- moved R10 81.3 mm to (36.0, 41.0)
- moved R9 67.8 mm to (99.0, 66.0)
- moved R17 61.1 mm to (40.0, 41.0)
- moved C51 57.6 mm to (91.0, 38.0)
- moved R14 56.6 mm to (81.0, 80.0)
- moved C44 55.4 mm to (91.0, 46.0)
- moved C54 52.6 mm to (40.0, 53.0)
- moved R11 52.6 mm to (62.0, 43.0)
- moved C52 51.2 mm to (91.0, 48.0)
- moved C47 47.9 mm to (44.0, 47.0)
- moved R25 47.0 mm to (81.0, 84.0)
- moved R26 47.0 mm to (85.0, 84.0)
- moved C45 45.3 mm to (89.0, 52.0)
- moved R27 43.6 mm to (79.0, 84.0)
- moved C46 35.4 mm to (36.0, 53.0)
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Connections:
- C31 pad 1: VBAT_MON -> VGND
- C31 pad 2: DGND -> AGND
- C32 pad 1: AVDD -> VGND
- C33 pad 1: AVDD -> VBAT_MON
- C33 pad 2: AGND -> DGND
- C42 pad 1: DVDD -> AVDD
- C42 pad 2: DGND -> AGND
- C43 pad 1: DVDD -> AVDD
- C43 pad 2: DGND -> AGND
- C54 pad 1: AVDD -> DVDD
- C54 pad 2: AGND -> DGND
- C55 pad 1: AVDD -> DVDD
- C55 pad 2: AGND -> DGND
- R10 pad 1: MUX2_X_OUT -> VBUS
- R10 pad 2: MUX1_X_FILT -> LED_STAT
- R11 pad 1: MUX2_Y_OUT -> LRCK_SRC
- R11 pad 2: MUX1_Y_FILT -> LRCK
- R12 pad 1: OUT_A_AC -> MCLK_SRC
- R12 pad 2: JACK_A_TIP -> MCLK
- R13 pad 1: OUT_B_AC -> MUX2_X_OUT
- R13 pad 2: JACK_B_TIP -> MUX1_X_FILT
- R14 pad 1: PROG_PIN -> MUX2_Y_OUT
- R14 pad 2: DGND -> MUX1_Y_FILT
- R15 pad 1: MUX1_X_OUT -> OUT_A_AC
- R15 pad 2: MUX1_X_FILT -> JACK_A_TIP
- R16 pad 1: MUX1_Y_OUT -> OUT_B_AC
- R16 pad 2: MUX1_Y_FILT -> JACK_B_TIP
- R17 pad 1: SIG_CH1 -> PROG_PIN
- R17 pad 2: SUM_FB_A -> DGND
- R18 pad 1: SIG_CH2 -> MUX1_X_OUT
- R18 pad 2: SUM_FB_A -> MUX1_X_FILT
- R19 pad 1: SIG_CH3 -> MUX1_Y_OUT
- R19 pad 2: SUM_FB_A -> MUX1_Y_FILT
- R20 pad 1: SIG_CH4 -> SIG_CH1
- R21 pad 1: SIG_CH5 -> SIG_CH2
- R21 pad 2: SUM_FB_B -> SUM_FB_A
- R22 pad 1: SIG_CH6 -> SIG_CH3
- R22 pad 2: SUM_FB_B -> SUM_FB_A
- R23 pad 1: SIG_CH7 -> SIG_CH4
- R23 pad 2: SUM_FB_B -> SUM_FB_A
- R24 pad 1: SIG_CH8 -> SIG_CH5
- R25 pad 1: DVDD -> SIG_CH6
- R25 pad 2: UART_SLAVE_TX -> SUM_FB_B
- R26 pad 1: VBAT_MON -> SIG_CH7
- R26 pad 2: DGND -> SUM_FB_B
- R27 pad 1: VBAT -> SIG_CH8
- R27 pad 2: VBAT_MON -> SUM_FB_B
- R7 pad 1: SUM_FB_A -> BCLK_SRC
- R7 pad 2: SUM_A -> BCLK
- R8 pad 1: SUM_FB_B -> SUM_FB_A
- R8 pad 2: SUM_B -> SUM_A
- R9 pad 1: VBUS -> SUM_FB_B
- R9 pad 2: LED_STAT -> SUM_B
- U1 pad 5: MCLK -> MCLK_SRC
- U1 pad 6: BCLK -> BCLK_SRC
- U1 pad 7: LRCK -> LRCK_SRC
- U12 pad 3: AGND -> VGND
- U12 pad 5: AGND -> VGND
Routing:
- net MUX_B: track 0.00 -> 39.1 mm, vias 0 -> 2
- net DGND: track 0.00 -> 39.0 mm, vias 0 -> 13
- net MUX_A: track 0.00 -> 35.1 mm, vias 0 -> 2
- net MUX_INH: track 0.00 -> 19.0 mm, vias 0 -> 2
- net MCLK: track 46.9 -> 34.2 mm
- net BCLK: track 41.0 -> 33.2 mm
- net LRCK: track 36.4 -> 33.4 mm
