File: boards/preamp/layout/layout.kicad_pcb (KiCad board)
At the start: 4 copper layers, 100 x 80 mm, 157 parts, among them J1 61300211121, J10 61300211121, J11 61300211121, J12 61300211121, J13 61300211121, J14 61300211121, J15 61300211121, J16 61300211121, J17 61301021121, J18 61300211121, J2 61300211121, J3 61300211121, J4 61300211121, J5 61300211121, J6 61300211121, J7 61300211121, J8 61300211121, J9 61300211121, U1 NE5532DR, U10 NE5532DR, U11 NE5532DR, U12 NE5532DR, U13 NE5532DR, U14 NE5532DR, U2 NE5532DR, U3 NE5532DR, U4 NE5532DR, U5 LP2985-33DBVR, U6 NE5532DR, U7 NE5532DR, U8 NE5532DR, U9 NE5532DR

Commit message: esp32 footprint, layout changes, removed charging usb
Parts:
- moved C30 88.4 mm to (31.0, 84.0)
- moved H2 85.3 mm to (22.0, 80.0)
- moved C28 77.7 mm to (21.0, 84.0)
- moved C31 77.7 mm to (79.0, 20.0)
- moved H1 67.0 mm to (15.0, 80.0)
- moved C58 63.5 mm to (35.0, 18.0)
- moved C26 58.1 mm to (55.0, 26.0)
- moved C34 56.9 mm to (75.0, 88.0)
- moved C67 56.5 mm to (35.0, 22.0)
- moved C53 51.0 mm to (35.0, 36.0)
- moved R2 51.0 mm to (99.0, 24.0)
- moved C32 50.4 mm to (41.0, 84.0)
- moved C62 48.1 mm to (45.0, 34.0)
- moved C49 46.7 mm to (45.0, 20.0)
- moved R8 41.2 mm to (99.0, 78.0)
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
Commit message: fixes
Parts:
- removed H1, H2: ?, MountingHole_3.2mm_M3_DIN965_Pad_TopBottom
- moved C30 80.0 mm to (79.0, 20.0)
- moved C28 77.7 mm to (65.0, 20.0)
- moved R35 60.9 mm to (105.0, 12.0)
- moved C2 59.9 mm to (99.0, 24.0)
- moved C34 56.9 mm to (39.0, 44.0)
- moved C1 51.3 mm to (103.0, 12.0)
- moved R1 47.1 mm to (103.0, 20.0)
- moved R8 47.1 mm to (53.0, 68.0)
- moved C41 42.9 mm to (71.0, 88.0)
- moved C37 42.4 mm to (79.0, 82.0)
- moved C39 40.5 mm to (69.0, 44.0)
- moved R3 35.4 mm to (69.0, 40.0)
- moved C24 33.5 mm to (49.0, 62.0)
- moved R37 33.0 mm to (71.0, 30.0)
- moved R6 31.0 mm to (99.0, 62.0)
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
Commit message: layout changes
Parts:
- moved C31 86.0 mm to (35.0, 84.0)
- moved C30 80.0 mm to (31.0, 84.0)
- moved C1 77.9 mm to (35.0, 50.0)
- moved C27 72.5 mm to (49.0, 20.0)
- moved C26 58.1 mm to (51.0, 84.0)
- moved R7 54.9 mm to (103.0, 74.0)
- moved R1 53.0 mm to (51.0, 30.0)
- moved C2 51.0 mm to (49.0, 34.0)
- moved R2 50.0 mm to (51.0, 40.0)
- moved C35 48.2 mm to (39.0, 56.0)
- moved C37 45.3 mm to (49.0, 48.0)
- moved R36 44.0 mm to (59.0, 30.0)
- moved R41 42.2 mm to (103.0, 66.0)
- moved C38 40.4 mm to (69.0, 44.0)
- moved C8 40.0 mm to (87.0, 44.0)
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